File: kicad project files/AS-MULTI-UNO-01/AS-MULTI-UNO-01.kicad_pcb (KiCad board)
At the start: 2 copper layers, 75.6 x 54 mm, 11 parts, among them J1 ICSP, J2 Conn_01x02, U1 ATmega328-P, Y1 12Mhz

Commit message: Update to version v1.2
Parts:
- added J3: Conn_01x06, Connector_PinHeader_2.54mm:PinHeader_1x06_P2.54mm_Horizontal, F.Cu at (134.8, 94.5)
- added SW1: SW_Push, Button_Switch_THT:SW_PUSH_6mm_H4.3mm, F.Cu at (136.8, 111.2)
Connections:
- net /RESET renamed /DTR
Routing:
- net /D0/RX: track 24.7 -> 97.0 mm, vias 0 -> 7
- net /D1/TX: track 24.7 -> 95.4 mm, vias 0 -> 7
- net /DTR: track 73.6 -> 112.9 mm
- net VCC: track 97.5 -> 120.3 mm
- net /D4: track 24.7 -> 25.5 mm
Other:
- board text added: "DTR"
- board text added: "RX"
- board text added: "SERIAL UART"
- board text added: "TX"
- board text added: "©Akerasoft 2022 AS-MULTI-UNO-01 V1.2 OPEN SOURCE NO VOLTAGE REGULATION"
- board text removed: "©Akerasoft 2022 AS-MULTI-UNO-01 V1.1 OPEN SOURCE NO VOLTAGE REGULATION"
