File: kicad project files/AS-MULTI-UNO-01/AS-MULTI-UNO-01.kicad_sch (KiCad schematic)
At the start: 11 parts, among them J1 ICSP, J2 Conn_01x02, U1 ATmega328-P, Y1 12Mhz

Commit message: Update to version v1.2
Parts:
- added J3: Conn_01x06, Connector_PinHeader_2.54mm:PinHeader_1x06_P2.54mm_Horizontal, symbol Connector_Generic:Conn_01x06
- added SW1: SW_Push, Button_Switch_THT:SW_PUSH_6mm_H4.3mm, symbol Switch:SW_Push
- J2: footprint (none) -> Connector_JST:JST_XH_S2B-XH-A_1x02_P2.50mm_Horizontal
Connections:
- net D0/RX: now also J3.3 (Pin_3)
- net D1/TX: now also J3.2 (Pin_2)
- net GND: now also J3.6 (Pin_6), SW1.2
- net VCC: now also J3.4 (Pin_4)
- net RESET renamed DTR
- net DTR: now also J3.1 (Pin_1), SW1.1
- new net CTS: J3.5 (Pin_5)
Other:
- note added: "NOT CONNECTED"
- note added: "RESET"
- note added: "RESET CIRCUIT"
- note added: "SERIAL RX"
- note added: "SERIAL TX"
- note added: "TRANSMIT AND RECEIVE NEED TO BE CROSSED"
- note added: "TTL SERIAL/UART"
- moved on the sheet: C3, C4, C5, R1
